Commit message: モデル追加

File: urdf/thouzer.urdf (robot description, URDF)
Before this commit: robot thouzer, 1 links, 0 joints
Links:
- link base_link: geometry collision mesh filename=package://thouzer_description/meshes/RMS-SZE2.STL scale=0.001 0.001 0.001; visual mesh filename=package://thouzer_description/meshes/RMS-SZE2.STL scale=0.001 0.001 0.001
